Commit message: Simulation Updates

File: description/properties.xacro (robot description, xacro)
@@ -14,4 +14,5 @@
   <xacro:property name="outer_ankle_joint_z" value="0.13653" />
   <xacro:property name="center_ankle_joint_z" value="0.12383" />
+  <xacro:property name="center_wheel_radius" value="0.0508" /> <!-- 4" diameter -->
   <xacro:property name="wheel_radius" value="0.059685" /><!-- 5cm radius -->
   <xacro:property name="wheel_thickness" value="0.05" /> <!-- 5cm -->

File: description/robot.urdf.xacro (robot description, xacro)
@@ -7,7 +7,9 @@
         <xacro:include filename="ros2_control.xacro" />
     </xacro:if>
+    <!--
     <xacro:unless value="$(arg use_ros2_control)">
         <xacro:include filename="gazebo_control.xacro" />
     </xacro:unless>
+    -->
     <!--
     <xacro:include filename="lidar.xacro" />

File: description/robot_core.xacro (robot description, xacro)
@@ -138,4 +138,28 @@
         <mu2>0</mu2>
     </gazebo>
+    <!-- LEFT FOOT LINK -->
+    <joint name="left_foot_joint" type="fixed">
+        <parent link="base_link"/>
+        <child link="left_foot"/>
+        <origin xyz="0 ${wheel_separation / 2} ${foot_distance_from_ground}"/>
+    </joint>
+    <link name="left_foot">
+        <visual>
+            <origin xyz="0 0 0" rpy="${radians(90)} 0 0" />
+            <geometry>
+                <mesh filename="package://r2_ros/meshes/left_foot.stl" scale="0.001 0.001 0.001" />
+            </geometry>
+            <material name="white" />
+        </visual>
+        <collision>
+            <origin xyz="0 0 0" rpy="${radians(90)} 0 0" />
+            <geometry>
+                <mesh filename="package://r2_ros/meshes/left_foot.stl" scale="0.001 0.001 0.001" />
+            </geometry>
+        </collision>
+        <xacro:inertial_box mass="${foot_mass}" x="${foot_length}" y="${foot_width}" z="${foot_height}">
+            <origin xyz="0 ${foot_width_offset} ${foot_height/2}" rpy="0 0 0"/>
+        </xacro:inertial_box>
+    </link>
     <!-- RIGHT FOOT LINK -->
     <joint name="right_foot_joint" type="fixed">
@@ -162,5 +186,30 @@
         </xacro:inertial_box>
     </link>
-    <!-- RIGHT ANGLE JOINT -->
+    <!-- LEFT ANKLE JOINT -->
+    <joint name="left_ankle_joint" type="revolute">
+        <origin xyz="0 -0.0425 ${outer_ankle_joint_z}" rpy="0 0 0" />
+        <parent link="left_foot" />
+        <child link="left_leg" />
+        <axis xyz="0 -1 0" />
+        <limit lower="-${radians(18)}" upper="${radians(2)}" velocity="100" effort="100" />
+    </joint>
+    <link name="left_leg">
+        <visual>
+            <origin xyz="0 0 0.5496052" rpy="${radians(180)} 0 ${radians(180)}" />
+            <geometry>
+                <mesh filename="package://r2_ros/meshes/left_leg.obj" scale="1 1 1" />
+            </geometry>
+        </visual>
+        <collision>
+            <origin xyz="0 0 0.5496052" rpy="${radians(180)} 0 ${radians(180)}" />
+            <geometry>
+                <mesh filename="package://r2_ros/meshes/left_leg.obj" scale="1 1 1" />
+            </geometry>
+        </collision>
+        <xacro:inertial_box mass="${leg_mass}" x="${leg_width}" y="${leg_depth}" z="${leg_length}">
+            <origin xyz="0 0.02215 ${leg_length / 2}" rpy="0 0 0"/>
+        </xacro:inertial_box>
+    </link>
+    <!-- RIGHT ANKLE JOINT -->
     <joint name="right_ankle_joint" type="revolute">
         <origin xyz="0 0.0425 ${outer_ankle_joint_z}" rpy="0 0 0" />
@@ -193,17 +242,32 @@
         ${0.5496052 - 0.245745 + 0.098425}
     -->
+    <!--
+    <joint name="left_shoulder_joint" type="revolute">
+        <origin xyz="0 ${body_radius - 0.0127} ${0.5496052}" rpy="0 0 0" />
+        <parent link="left_leg" />
+        <child link="shoulder" />
+        <axis xyz="0 -1 0" />
+        <limit lower="-${radians(4)}" upper="${radians(36)}" velocity="100" effort="100" />
+    </joint>
+    -->
     <joint name="right_shoulder_joint" type="revolute">
         <origin xyz="0 ${body_radius + 0.0127} ${0.5496052}" rpy="0 0 0" />
         <parent link="right_leg" />
+        <child link="shoulder" />
+        <axis xyz="0 -1 0" />
+        <limit lower="-${radians(4)}" upper="${radians(36)}" velocity="100" effort="100" />
+    </joint>
+    <link name="shoulder">
+    </link>
+    <xacro:property name="body_mass" value="1"/>
+    <joint name="shoulder_link" type="fixed">
+        <origin xyz="0 0 0" rpy="0 0 0" />
+        <parent link="shoulder" />
         <child link="body" />
-        <axis xyz="0 -1 0" />
-        <limit lower="-${radians(4)}" upper="${radians(36)}" velocity="100" effort="100" />
-    </joint>
-    <xacro:property name="body_mass" value="1"/>
+    </joint>
     <link name="body">
         <visual>
             <origin xyz="0 0 ${body_shoulder_offset}" rpy="${radians(90)} 0 ${radians(90)}" />
             <geometry>
-                <!--<cylinder length="${body_height}" radius="${body_radius}" /> -->
                 <!-- Exported in meters -->
                 <mesh filename="package://r2_ros/meshes/frame.obj" scale="1 1 1" />
@@ -219,57 +283,4 @@
             <origin xyz="0 0 ${body_shoulder_offset - (body_height/2)}" rpy="0 0 0"/>
         </xacro:inertial_cylinder>
-    </link>
-    <!-- LEFT SHOULDER & LEG -->
-    <joint name="left_shoulder_joint" type="revolute">
-        <origin xyz="0 ${body_radius + 0.0127} 0" rpy="0 0 ${radians(180)}" />
-        <parent link="body" />
-        <child link="left_leg" />
-        <axis xyz="0 -1 0" />
-        <limit lower="-${radians(4)}" upper="${radians(36)}" velocity="100" effort="100" />
-        <mimic joint="right_shoulder_joint" multiplier="1" offset="0" />
-    </joint>
-    <link name="left_leg">
-        <visual>
-            <origin xyz="0 0 0" rpy="${radians(180)} 0 0" />
-            <geometry>
-                <mesh filename="package://r2_ros/meshes/left_leg.obj" scale="1 1 1" />
-            </geometry>
-        </visual>
-        <collision>
-            <origin xyz="0 0 0" rpy="${radians(180)} 0 0" />
-            <geometry>
-                <mesh filename="package://r2_ros/meshes/left_leg.obj" scale="1 1 1" />
-            </geometry>
-        </collision>
-        <xacro:inertial_box mass="${leg_mass}" x="${leg_width}" y="${leg_depth}" z="${leg_length}">
-            <origin xyz="0 -0.02215 ${-leg_length / 2}" rpy="0 0 0"/>
-        </xacro:inertial_box>
-    </link>
-    <!-- LEFT ANKLE & FOOT -->
-    <joint name="left_ankle_joint" type="revolute">
-        <origin xyz="0 -0.0425 -${0.5496052}" rpy="0 0 0" />
-        <parent link="left_leg" />
-        <child link="left_foot" />
-        <axis xyz="0 -1 0" />
-        <limit lower="-${radians(18)}" upper="${radians(2)}" velocity="100" effort="100" />
-        <mimic joint="right_ankle_joint" multiplier="1" offset="0" />
-    </joint>
-    <link name="left_foot">
-        <visual>
-            <origin xyz="0 0 ${-outer_ankle_joint_z}" rpy="${radians(90)} 0 ${radians(180)}" />
-            <geometry>
-                <mesh filename="package://r2_ros/meshes/left_foot.stl" scale="0.001 0.001 0.001" />
-            </geometry>
-            <material name="white" />
-        </visual>
-        <collision>
-            <origin xyz="0 0 ${-outer_ankle_joint_z}" rpy="${radians(90)} 0 ${radians(180)}" />
-            <geometry>
-                <mesh filename="package://r2_ros/meshes/left_foot.stl" scale="0.001 0.001 0.001" />
-            </geometry>
-        </collision>
-        <xacro:inertial_box mass="${foot_mass}" x="${foot_length}" y="${foot_width}" z="${foot_height}">
-            <origin xyz="0 ${foot_width_offset} ${0.01725-(foot_height/2)}" rpy="0 0 0"/>
-        </xacro:inertial_box>
     </link>
     <!-- CENTER LEG -->
@@ -304,5 +315,7 @@
         <axis xyz="0 -1 0" />
         <limit lower="-${radians(18)}" upper="${radians(2)}" velocity="100" effort="100" />
-        <mimic joint="right_ankle_joint" multiplier="1" offset="0" />
+        <xacro:unless value="$(arg sim_mode)">
+            <mimic joint="right_ankle_joint" multiplier="1" offset="0" />
+        </xacro:unless>
     </joint>
     <link name="center_foot">
@@ -328,5 +341,5 @@
         <parent link="center_foot"/>
         <child link="center_front_idler"/>
-        <origin xyz="${front_wheel_offset} 0 -${center_ankle_joint_z - wheel_radius + foot_distance_from_ground}" rpy="${pi/2} 0 0" />
+        <origin xyz="-${center_wheel_radius + 0.01} 0 -${center_ankle_joint_z - center_wheel_radius + foot_distance_from_ground}" rpy="${pi/2} 0 0" />
         <axis xyz="0 0 -1"/>
     </joint>
@@ -334,18 +347,45 @@
         <visual>
             <geometry>
-                <cylinder radius="${wheel_radius}" length="${wheel_thickness}"/>
-            </geometry>
-            <material name="blue"/>
-        </visual>
-        <collision>
-            <geometry>
-                <cylinder radius="${wheel_radius}" length="${wheel_thickness}"/>
-            </geometry>
-        </collision>
-        <xacro:inertial_cylinder mass="${wheel_mass}" length="${wheel_thickness}" radius="${wheel_radius}">
+                <cylinder radius="${center_wheel_radius}" length="${wheel_thickness}"/>
+            </geometry>
+            <material name="blue"/>
+        </visual>
+        <collision>
+            <geometry>
+                <cylinder radius="${center_wheel_radius}" length="${wheel_thickness}"/>
+            </geometry>
+        </collision>
+        <xacro:inertial_cylinder mass="${wheel_mass}" length="${wheel_thickness}" radius="${center_wheel_radius}">
             <origin xyz="0 0 0" rpy="0 0 0"/>
         </xacro:inertial_cylinder>
     </link>
     <gazebo reference="center_front_idler">
+        <material>Gazebo/Blue</material>
+        <mu1>0</mu1>
+        <mu2>0</mu2>
+    </gazebo>
+    <joint name="center_rear_idler_joint" type="continuous">
+        <parent link="center_foot"/>
+        <child link="center_rear_idler"/>
+        <origin xyz="${center_wheel_radius + 0.01} 0 -${center_ankle_joint_z - center_wheel_radius + foot_distance_from_ground}" rpy="${pi/2} 0 0" />
+        <axis xyz="0 0 -1"/>
+    </joint>
+    <link name="center_rear_idler">
+        <visual>
+            <geometry>
+                <cylinder radius="${center_wheel_radius}" length="${wheel_thickness}"/>
+            </geometry>
+            <material name="blue"/>
+        </visual>
+        <collision>
+            <geometry>
+                <cylinder radius="${center_wheel_radius}" length="${wheel_thickness}"/>
+            </geometry>
+        </collision>
+        <xacro:inertial_cylinder mass="${wheel_mass}" length="${wheel_thickness}" radius="${center_wheel_radius}">
+            <origin xyz="0 0 0" rpy="0 0 0"/>
+        </xacro:inertial_cylinder>
+    </link>
+    <gazebo reference="center_rear_idler">
         <material>Gazebo/Blue</material>
         <mu1>0</mu1>

File: description/ros2_control.xacro (robot description, xacro)
@@ -52,4 +52,41 @@
                 <state_interface name="position"/>
             </joint>
+            <joint name="left_ankle_joint">
+                <command_interface name="position">
+                    <param name="min">-${radians(18)}</param>
+                    <param name="max">${radians(2)}</param>
+                </command_interface>
+                <state_interface name="velocity" />
+                <state_interface name="position" />
+            </joint>
+            <joint name="right_ankle_joint">
+                <command_interface name="position">
+                    <param name="min">-${radians(18)}</param>
+                    <param name="max">${radians(2)}</param>
+                </command_interface>
+                <state_interface name="velocity" />
+                <state_interface name="position" />
+            </joint>
+            <joint name="right_shoulder_joint">
+                <command_interface name="position">
+                    <param name="min">-${radians(4)}</param>
+                    <param name="max">${radians(36)}</param>
+                </command_interface>
+                <state_interface name="velocity" />
+                <state_interface name="position" />
+            </joint>
+            <joint name="center_foot_joint">
+                <command_interface name="position">
+                    <param name="min">-${radians(18)}</param>
+                    <param name="max">${radians(2)}</param>
+                </command_interface>
+                <state_interface name="velocity" />
+                <state_interface name="position" />
+            </joint>
+            <joint name="dome_joint">
+                <command_interface name="position" />
+                <state_interface name="velocity" />
+                <state_interface name="position" />
+            </joint>
         </ros2_control>
     </xacro:if>
