Commit message: Latest State

File: description/robot_core.xacro (robot description, xacro)
@@ -242,13 +242,13 @@
         ${0.5496052 - 0.245745 + 0.098425}
     -->
-    <!--
-    <joint name="left_shoulder_joint" type="revolute">
-        <origin xyz="0 ${body_radius - 0.0127} ${0.5496052}" rpy="0 0 0" />
-        <parent link="left_leg" />
-        <child link="shoulder" />
-        <axis xyz="0 -1 0" />
-        <limit lower="-${radians(4)}" upper="${radians(36)}" velocity="100" effort="100" />
-    </joint>
-    -->
+    <xacro:unless value="$(arg sim_mode)">
+        <joint name="left_shoulder_joint" type="revolute">
+            <origin xyz="0 ${body_radius - 0.0127} ${0.5496052}" rpy="0 0 0" />
+            <parent link="left_leg" />
+            <child link="shoulder" />
+            <axis xyz="0 -1 0" />
+            <limit lower="-${radians(4)}" upper="${radians(36)}" velocity="100" effort="100" />
+        </joint>
+    </xacro:unless>
     <joint name="right_shoulder_joint" type="revolute">
         <origin xyz="0 ${body_radius + 0.0127} ${0.5496052}" rpy="0 0 0" />

File: description/ros2_control.xacro (robot description, xacro)
@@ -2,4 +2,7 @@
 <robot xmlns:xacro="http://www.ros.org/wiki/xacro">
     <xacro:unless value="$(arg sim_mode)">
+        <ros2_control name="RealRobot" type="generic_system">
+        </ros2_control>
+    <!--
         <ros2_control name="RealRobot" type="system">
             <hardware>
@@ -30,4 +33,5 @@
             </joint>
         </ros2_control>
+        -->
     </xacro:unless>
     <xacro:if value="$(arg sim_mode)">
